File: PCB/Main Boards/OSO-SWAT-C1/OSO-SWAT-C1.kicad_sch (KiCad schematic)
At the start: 35 parts, among them J1 OSO_SWD, J2 FH19C-9S-0.5SH_10_, Q1 Q_Photo_NPN, Q2 Q_NMOS_GSD, U1 ATSAML22J18A-MUT, U2 MIC5365-3.3YC5-TR, X1 Crystal

Commit message: Initial commit.
Parts:
- removed C1: 10uF, Capacitor_SMD:C_0603_1608Metric, symbol OSO-SWAT-A1-05-eagle-import:CAP_CERAMIC_0603MP
- removed C2: 0.1uF, Capacitor_SMD:C_0201_0603Metric, symbol OSO-SWAT-A1-05-eagle-import:CAP_CERAMIC_0603MP
- removed C3, C4: 0.1uF, Capacitor_SMD:C_0603_1608Metric, symbol OSO-SWAT-A1-05-eagle-import:CAP_CERAMIC_0603MP
- removed C5, C6, C9: 1uF, Capacitor_SMD:C_0603_1608Metric, symbol OSO-SWAT-A1-05-eagle-import:CAP_CERAMIC_0603MP
- removed C7, C8: 22pf, Capacitor_SMD:C_0402_1005Metric, symbol OSO-SWAT-A1-05-eagle-import:CAP_CERAMIC_0402MP
- removed D1: SCHOTTKY, OSO-SWAT-A1-05:SOD-323F, symbol OSO-SWAT-A1-05-eagle-import:DIODESOD-323F
- removed J1: OSO_SWD, OSO-SWD:OSO_SWD_2x3, symbol OSO-SWD:OSO_SWD
- removed J2: FH19C-9S-0.5SH_10_, OSO-SWAT-A1-05:FH19C9S05SH10, symbol OSO-SWAT-A1-05-eagle-import:FH19C-9S-0.5SH_10_
- removed L1: 10uH, Inductor_SMD:L_0805_2012Metric, symbol OSO-SWAT-A1-05-eagle-import:MICROBUILDER_INDUCTOR_0805MP
- removed L2: 14 mH, OSO-SWAT-A1-05:ELT3KN, symbol OSO-SWAT-A1-05-eagle-import:MICROBUILDER_INDUCTOR_0805MP
- removed R1, R3, R4: 10K, Resistor_SMD:R_0201_0603Metric, symbol OSO-SWAT-A1-05-eagle-import:RESISTOR_0603MP
- removed R10: 10K THERM, Resistor_SMD:R_0603_1608Metric, symbol OSO-SWAT-A1-05-eagle-import:RESISTOR_0603MP
- removed R11: 10K 0.1%, Resistor_SMD:R_0603_1608Metric, symbol OSO-SWAT-A1-05-eagle-import:RESISTOR_0603MP
- removed R2: 10K, Resistor_SMD:R_0201_0603Metric, symbol Device:R
- removed R6: 1K, Resistor_SMD:R_0603_1608Metric, symbol OSO-SWAT-A1-05-eagle-import:RESISTOR_0603MP
- removed R7, R8: 100, Resistor_SMD:R_0603_1608Metric, symbol OSO-SWAT-A1-05-eagle-import:RESISTOR_0603MP
- removed TP1, TP10, TP8, TP9: MICROBUILDER_TESTPOINTROUND1.5MM, OSO-SWAT-A1-05:MICROBUILDER_TESTPOINT_ROUND_1.5MM, symbol OSO-SWAT-A1-05-eagle-import:MICROBUILDER_TESTPOINTROUND1.5MM
- removed U1: ATSAML22J18A-MUT, OSO-SWAT-A1-05:QFN64_9X9MC_MCH, symbol OSO-SWAT-A1-05-eagle-import:ATSAML22J18A-MUT
- removed U2: MIC5365-3.3YC5-TR, OSO-SWAT-A1-05:SOT65P210X110-5N, symbol OSO-SWAT-A1-05-eagle-import:MIC5365-3.3YC5-TR
- removed X1: Crystal, Crystal:Crystal_SMD_3215-2Pin_3.2x1.5mm, symbol Device:Crystal
- added AE1: amemb-2450AT42E0100, amemb-RF_Antenna.pretty:amemb-2450AT42E0100, symbol amemb-RF_Antenna:amemb-2450AT42E0100
- added BZ1: Buzzer, OSO-SWAT-A1-05:ELT3KN, symbol Device:Buzzer
- added C1, C2: TBD, passives:C_0201_0603Metric_L, symbol Device:C_Small
- added C10, C11, C12, C13, C14, C16, C17, C4, C46, C47, C48, C49, C5, C50, C51, C7, C8, C9: 1uF, passives:C_0201_0603Metric_L, symbol Device:C_Small
- added C15, C6: 10uF, passives:C_0402_1005Metric_L, symbol Device:C_Small
- added C3: 220nF, passives:C_0201_0603Metric_L, symbol Device:C_Small
- added J3: Conn_ARM_SWD_TagConnect_TC2030-NL, Connector:Tag-Connect_TC2030-IDC-NL_2x03_P1.27mm_Vertical, symbol Connector:Conn_ARM_SWD_TagConnect_TC2030-NL
- added J4: Conn_02x05_Odd_Even_MountingPin, Connector_Hirose_DF40:Hirose_DF40B-10DS-0.4V_2x05-1MP_P0.4mm, symbol Connector_Generic_MountingPin:Conn_02x05_Odd_Even_MountingPin
- added L1: 0R, passives:R_0201_0603Metric_L, symbol Device:L_Small
- added Q3: Q_NMOS_GSD, Package_DFN_QFN:Diodes_DFN1006-3, symbol Device:Q_NMOS_GSD
- added R1: 10kR, passives:R_0201_0603Metric_L, symbol Device:R_Small_US
- added R10, R11, R9: 100kR, passives:R_0201_0603Metric_L, symbol Device:R_Small_US
- added R3: 100kR, 0.1%, passives:R_0201_0603Metric_L, symbol Device:R_Small_US
- added R4, R6: 100R, passives:R_0201_0603Metric_L, symbol Device:R_Small_US
- added R5: 1kR, passives:R_0201_0603Metric_L, symbol Device:R_Small_US
- added R7, R8: 5.1kR, passives:R_0201_0603Metric_L, symbol Device:R_Small_US
- added TH1: 100kR, passives:R_0201_0603Metric_L, symbol Device:Thermistor_US
- added TP1, TP2: TestPoint, amemb-TestPoint.pretty:TestPoint_Pad_1.0x1.0mm_No_Silk, symbol Connector:TestPoint
- added U1: NCP115AMX250TCG, Package_DFN_QFN:OnSemi_XDFN4-1EP_1.0x1.0mm_EP0.52x0.52mm, symbol Regulator_Linear:NCP115AMX250TCG
- added U10: TPS22991, amemb-easyeda.pretty:4-UQFN-0.9x0.8mm, symbol amemb-Power_Management:TPS22991
- added U2: ADXL367, amemb-Package_LGA.pretty:amemb-ADXL367_LGA-12_2.11x2.21mm_P0.5mm_LayoutBorder2x4y, symbol amemb-Sensor_Motion:ADXL367
- added U3: HJ-N54L_SIP, easyeda2kicad:COMM-SMD_L4.5-W4.5-P0.55-S0.55-TR, symbol amemb-RF_Module:HJ-N54L_SIP
- added U4: BU97930MUV-E2, Package_DFN_QFN:VQFN-40-1EP_6x6mm_P0.5mm_EP3.5x3.5mm, symbol easyeda2kicad:BU97930MUV-E2
- added U5: W25Q128JVE, Package_SON:Winbond_USON-8-1EP_3x2mm_P0.5mm_EP0.2x1.6mm, symbol Memory_Flash:W25Q128JVE
- added U6: TPS22991, amemb-Package_DFN_QFN.pretty:4-UQFN-0.9x0.8mm, symbol amemb-Power_Management:TPS22991
- added U7: STM32L052T8Yx, Package_CSP:ST_WLCSP-36_Die417, symbol MCU_ST_STM32L0:STM32L052T8Yx
- added U8: TXU0204RUTR, amemb-Package_DFN_QFN.pretty:UQFN-12_L2.0-W1.7-P0.40-TL, symbol amemb-Logic_LevelTranslator:TXU0204RUTR
- added U9: TXU0101DRYR, amemb-Package_SON.pretty:SON-6_L1.5-W1.0-P0.50-TL, symbol amemb-Logic_LevelTranslator:TXU0101DRYR
- Q1: footprint Resistor_SMD:R_0603_1608Metric -> Diode_SMD:D_0603_1608Metric
- Q2: footprint Package_TO_SOT_SMD:SOT-523 -> Package_DFN_QFN:Diodes_DFN1006-3
- U$2: now in the parts list
Connections:
- net ALARM: now also U3.1 (P0.00)
- net BUZZER: now also R9.1, U3.7 (P1.07)
- net BUZZER_HV: now also BZ1.2 (-)
- net COM0: now also U4.8 (COM0)
- net COM1: now also U4.9 (COM1)
- net COM2: now also U4.10 (COM2)
- net GND: now also AE1.3 (GND), AE1.4 (GND), C1.2, C10.2, C11.2, C12.2, C13.2, C14.2, C15.2, C16.2, C17.2, C2.2, C3.2, C4.2, C46.2, C47.2, C48.2, C49.2, C5.2, C50.2, C51.2, C6.2, C7.2, C8.2, C9.2, J3.5 (GND), J4.2 (Pin_2), J4.7 (Pin_7), J4.8 (Pin_8), J4.9 (Pin_9), J4.MP (MountPin), Q3.2 (S), R10.2, R11.2, R7.1, R8.1, R9.2, U1.2 (GND), U1.5 (GND), U10.4 (GND), U2.11 (GND), U2.7 (GND), U3.[19,22,25,39] (GND), U4.[40,41] (VSS), U5.4 (GND), U5.9 (EP), U6.4 (GND), U7.D6 (VSS), U8.6 (GND), U9.2 (GND)
- net LIGHTSENSE: now also R1.2
- net SCL: now also J4.3 (Pin_3), U3.17 (P1.12)
- net SDA: now also J4.5 (Pin_5), U3.14 (P1.13)
- net SEG0: now also U4.12 (SEG0)
- net SEG1: now also U4.13 (SEG1)
- net SEG10: now also U4.22 (SEG10)
- net SEG11: now also U4.23 (SEG11)
- net SEG12: now also U4.24 (SEG12)
- net SEG13: now also U4.25 (SEG13)
- net SEG14: now also U4.26 (SEG14)
- net SEG15: now also U4.27 (SEG15)
- net SEG16: now also U4.28 (SEG16)
- net SEG17: now also U4.29 (SEG17)
- net SEG18: now also U4.30 (SEG18)
- net SEG19: now also U4.31 (SEG19)
- net SEG2: now also U4.14 (SEG2)
- net SEG20: now also U4.32 (SEG20)
- net SEG21: now also U4.33 (SEG21)
- net SEG22: now also U4.34 (SEG22)
- net SEG23: now also U4.35 (SEG23)
- net SEG3: now also U4.15 (SEG3)
- net SEG4: now also U4.16 (SEG4)
- net SEG5: now also U4.17 (SEG5)
- net SEG6: now also U4.18 (SEG6)
- net SEG7: now also U4.19 (SEG7)
- net SEG8: now also U4.20 (SEG8)
- net SEG9: now also U4.21 (SEG9)
- net TEMPSENSE: now also R3.1, TH1.2, U2.8 (ADC_{IN})
- net VBUS: now also C8.1, R10.1, U1.3 (EN), U1.4 (IN)
- net ~{BLUE}: now also R4.2, U3.9 (P1.06)
- net ~{GREEN}: now also R5.2, U3.11 (P1.05)
- net ~{LS_ENABLE}: now also U3.41 (P2.09)
- net ~{RED}: now also R6.2, U3.33 (P1.04)
- net ~{RESET}: now also J3.3 (~{RESET}), Q3.3 (D), U3.37 (~{RESET})
- net ~{TS_ENABLE}: now also R3.2, U3.3 (P2.10)
- net at D2.4 (CG): now also R5.1
- net at D2.3 (CB): now also R4.1
- net at D2.1 (CR): now also R6.1
- net SWCLK_LIGHT renamed LIGHT
- net LIGHT: now also U3.27 (P0.01)
- net SWDIO_MODE renamed MODE
- net MODE: now also U3.40 (P0.02)
- net USB_N renamed D-
- net D-: now also U7.C2 (PA11)
- net USB_P renamed D+
- net D+: now also U7.B1 (PA12)
- net VCC renamed VDD
- net VDD: now also BZ1.1 (+), C10.1, C11.1, C12.1, C14.1, C4.1, C46.1, C5.1, C6.1, C7.1, J3.1 (VCC), R1.1, TH1.1, U10.1 (VIN), U2.10 (V_{S}), U2.12 (V_{DDIO}), U3.[42-45] (VDD), U4.4 (VDD), U4.7 (VLCD), U5.8 (VCC), U6.1 (VIN)
- new net: R7.2, U$2.CC1
- new net: C13.1, J4.1 (Pin_1), U6.3 (VOUT)
- new net: J3.2 (SWDIO), U3.2 (SWDIO)
- new net: J3.4 (SWCLK), U3.28 (SWDCLK)
- new net: Q3.1 (G), R11.1, U7.C1 (PA10)
- new net: AE1.1 (FEED), C2.1, L1.2
- new net: R8.2, U$2.CC2
- new net: C1.1, L1.1, U3.23 (RF)
- new net: TP2.1, U3.30 (P1.03)
- new net: TP1.1, U3.8 (P1.02)
- new net: C3.1, U2.9 (V_{REG_OUT})
- new net DBG_SWCLK: U7.A1 (PA13), U8.2 (A1)
- new net DBG_SWDIO_IN: U7.A4 (PB7), U8.5 (A4Y)
- new net DBG_SWDIO_OE: U7.A3 (PB4), U9.5 (OE)
- new net DBG_SWDIO_OUT: U7.A2 (PA15), U9.3 (A)
- new net DEBUG.RX: U7.F5 (PA3), U8.4 (A3Y)
- new net DEBUG.TX: U7.E5 (PA2), U8.3 (A2)
- new net EN: U4.5 (EN)
- new net EN.EXT: U3.26 (P0.03), U6.2 (ON)
- new net GPIO.EXT: J4.10 (Pin_10), U3.31 (P1.15)
- new net LEVEL_SHIFT_VDD: C47.1, C48.1, C51.1, U10.3 (VOUT), U8.11 (VCCB), U9.6 (VCCB)
- new net MOSI: U3.36 (P1.09), U4.3 (MOSI)
- new net PDM.CLK: J4.4 (Pin_4), U3.15 (P1.11)
- new net PDM.DIN: J4.6 (Pin_6), U3.32 (P1.14)
- new net QSPI.D0: U3.13 (P2.02), U5.5 (DI/IO_{0})
- new net QSPI.D1: U3.38 (P2.04), U5.2 (DO/IO_{1})
- new net QSPI.D2: U3.35 (P2.03), U5.3 (~{WP}/IO_{2})
- new net QSPI.D3: U3.5 (P2.00), U5.7 (~{HOLD}/~{RESET}/IO_{3})
- new net QSPI.SCK: U3.6 (P2.01), U5.6 (CLK)
- new net QSPI.~{CS}: U3.4 (P2.05), U5.1 (~{CS})
- new net RX: U3.21 (P2.07), U8.9 (B2Y)
- new net SCK: U3.10 (P1.08), U4.2 (SCK)
- new net TARGET_SWDCLK: U8.10 (B1Y)
- new net TARGET_SWDIO: U8.7 (B4), U9.4 (BY)
- new net TX: U3.16 (P2.08), U8.8 (B3)
- new net VDD_DEBUGGER: C15.1, C16.1, C17.1, C49.1, C50.1, C9.1, U1.1 (OUT), U10.2 (ON), U7.A5 (VDD), U7.D5 (VDDA), U7.F1 (VDD), U8.1 (VCCA), U8.12 (OE), U9.1 (VCCA)
- new net ~{CS}: U3.18 (P1.10), U4.1 (~{CS})
- no-connect marks 1 -> 12
Other:
- note removed: "--LOCKED--"
- note removed: "Based on: arm-watch by @gregdavill, GoodWatch by @travisgoodspeed, and Pluto by Lukas K / carrotIndustries"
- note removed: "HS"
- note removed: "SERCOM0: IrDA SERCOM1: I2C SERCOM2: ? SERCOM3: SPI"
- note removed: "WO[4]"
- note removed: "WO[5]"
- note removed: "WO[6]"
- note removed: "WO[7]"
- moved on the sheet: D2A, D2B, D2C, Q1, Q2, RESET0, U$2A, U$2B
